Commit message: Added ros2 control support

File: bumperbot_description/urdf/bumperbot.urdf.xacro (robot description, xacro)
@@ -3,4 +3,5 @@
   <!-- Include Gazebo Parameters -->
   <xacro:include filename="$(find bumperbot_description)/urdf/bumperbot_gazebo.xacro" />
+  <xacro:include filename="$(find bumperbot_description)/urdf/bumperbot_ros2_control.xacro" />
   <link name="base_footprint"/>
   <link name="base_link">

File: bumperbot_description/urdf/bumperbot_gazebo.xacro (robot description, xacro)
@@ -1,4 +1,18 @@
 <?xml version="1.0"?>
 <robot name="bumperbot" xmlns:xacro="http://ros.org/wiki/xacro">
+  <transmission name="wheel_right_transmission">
+    <plugin>transmission_interface/SImpleTransmission</plugin>
+    <actuator name="wheel_right_motor" roll="actuator_right"/>
+    <joint name="wheel_right_joint" roll="joint_right">
+      <mechanical_reduction>1.0</mechanical_reduction>
+    </joint>
+  </transmission>
+  <transmission name="wheel_left_transmission">
+    <plugin>transmission_interface/SImpleTransmission</plugin>
+    <joint name="wheel_left_joint" roll="joint_left">
+      <mechanical_reduction>1.0</mechanical_reduction>
+    </joint>
+    <actuator name="wheel_left_motor" roll="actuator_left"/>
+  </transmission>
   <gazebo reference="wheel_right_link">
     <mu1>100000000000000.0</mu1>
@@ -35,3 +49,10 @@
     <minVel>0.1</minVel>
   </gazebo>
+  <gazebo>
+    <plugin filename="libgazebo_ros2_control.so" name="gazebo_ros2_control">
+      <robot_param>robot_description</robot_param>
+      <robot_param_node>robot_state_publisher</robot_param_node>
+      <parameters></parameters>
+    </plugin>
+  </gazebo>
 </robot>
